File: hardware/iosefka_motherboard/filter_and_vca.kicad_sch (KiCad schematic)
At the start: 92 parts, among them J1 Audio Out, J3 Audio In, J5 Conn_01x10, J6 Conn_01x10, J7 Conn_01x08, J8 Conn_01x08, Q1 2N3906, Q2 2N3906, U11 TL074, U12 TL074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

Commit message: parameter adjustments
Parts:
- C15, C25, C30, C36, C8: value 4.7u BP -> 4.7u NP; footprint Capacitor_THT:CP_Radial_D5.0mm_P2.50mm -> values_not_refs:CP_Radial_D6.3mm_P2.50mm_VALUE
- C9: footprint Capacitor_THT:CP_Radial_D5.0mm_P2.50mm -> values_not_refs:CP_Radial_D6.3mm_P2.50mm_VALUE
- Q1, Q2: footprint Package_TO_SOT_THT:TO-92_Inline_Wide -> values_not_refs:TO-92_Inline_Wide
- R27: value 1M -> DNP
- R35, R37: value 30k -> 15k
- R36: value 15k -> 7.5k
Changed lines of the file:
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@@
 			)
 		)
-		(property "Value" "4.7u BP"
+		(property "Value" "4.7u NP"
 			(at 39.37 22.86 90)
 			(effects
@@
 			)
 		)
-		(property "Footprint" "Capacitor_THT:CP_Radial_D5.0mm_P2.50mm"
+		(property "Footprint" "values_not_refs:CP_Radial_D6.3mm_P2.50mm_VALUE"
 			(at 43.18 18.0848 0)
 			(effects
@@
 			)
 		)
-		(property "Footprint" "Package_TO_SOT_THT:TO-92_Inline_Wide"
+		(property "Footprint" "values_not_refs:TO-92_Inline_Wide"
 			(at 156.21 78.105 0)
 			(effects
@@
 			)
 		)
-		(property "Footprint" "Package_TO_SOT_THT:TO-92_Inline_Wide"
+		(property "Footprint" "values_not_refs:TO-92_Inline_Wide"
 			(at 157.48 111.125 0)
 			(effects
@@
 			)
 		)
-		(property "Value" "1M"
+		(property "Value" "DNP"
 			(at 119.634 68.326 90)
 			(effects
@@
 			)
 		)
-		(property "Value" "30k"
+		(property "Value" "15k"
 			(at 192.278 91.186 90)
 			(effects
@@
 			)
 		)
-		(property "Value" "30k"
+		(property "Value" "15k"
 			(at 192.278 83.566 90)
 			(effects
@@
 			)
 		)
-		(property "Value" "4.7u BP"
+		(property "Value" "4.7u NP"
 			(at 39.37 34.29 90)
 			(effects
@@
 			)
 		)
-		(property "Footprint" "Capacitor_THT:CP_Radial_D5.0mm_P2.50mm"
+		(property "Footprint" "values_not_refs:CP_Radial_D6.3mm_P2.50mm_VALUE"
 			(at 43.18 29.5148 0)
 			(effects
@@
 			)
 		)
-		(property "Value" "15k"
+		(property "Value" "7.5k"
 			(at 192.278 87.376 90)
 			(effects
@@
 			)
 		)
-		(property "Value" "4.7u BP"
+		(property "Value" "4.7u NP"
 			(at 39.116 165.354 90)
 			(effects
@@
 			)
 		)
-		(property "Footprint" "Capacitor_THT:CP_Radial_D5.0mm_P2.50mm"
+		(property "Footprint" "values_not_refs:CP_Radial_D6.3mm_P2.50mm_VALUE"
 			(at 43.18 167.9448 0)
 			(effects
@@
 			)
 		)
-		(property "Footprint" "Capacitor_THT:CP_Radial_D5.0mm_P2.50mm"
+		(property "Footprint" "values_not_refs:CP_Radial_D6.3mm_P2.50mm_VALUE"
 			(at 39.37 138.43 0)
 			(effects
@@
 			)
 		)
-		(property "Value" "4.7u BP"
+		(property "Value" "4.7u NP"
 			(at 99.06 180.34 90)
 			(effects
@@
 			)
 		)
-		(property "Footprint" "Capacitor_THT:CP_Radial_D5.0mm_P2.50mm"
+		(property "Footprint" "values_not_refs:CP_Radial_D6.3mm_P2.50mm_VALUE"
 			(at 102.87 183.1848 0)
 			(effects
@@
 			)
 		)
-		(property "Value" "4.7u BP"
+		(property "Value" "4.7u NP"
 			(at 101.6 166.37 90)
 			(effects
@@
 			)
 		)
-		(property "Footprint" "Capacitor_THT:CP_Radial_D5.0mm_P2.50mm"
+		(property "Footprint" "values_not_refs:CP_Radial_D6.3mm_P2.50mm_VALUE"
 			(at 105.41 169.2148 0)
 			(effects
