File: hardware/iosefka_motherboard/power_supply.kicad_sch (KiCad schematic)
At the start: 14 parts, among them J2 DC In, U1 LM7805_TO220, U2 LM7905_TO220, U3 LT1054

Commit message: parameter adjustments
Parts:
- C1, C16, C20: footprint Capacitor_THT:CP_Radial_D5.0mm_P2.50mm -> values_not_refs:CP_Radial_D6.3mm_P2.50mm_VALUE
- C17, C2: footprint Capacitor_THT:CP_Radial_D6.3mm_P2.50mm -> values_not_refs:CP_Radial_D8.0mm_P2.50mm_VALUE
Changed lines of the file:
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@@
 			)
 		)
-		(property "Footprint" "Capacitor_THT:CP_Radial_D5.0mm_P2.50mm"
+		(property "Footprint" "values_not_refs:CP_Radial_D6.3mm_P2.50mm_VALUE"
 			(at 82.55 109.22 0)
 			(effects
@@
 			)
 		)
-		(property "Footprint" "Capacitor_THT:CP_Radial_D6.3mm_P2.50mm"
+		(property "Footprint" "values_not_refs:CP_Radial_D8.0mm_P2.50mm_VALUE"
 			(at 157.48 102.87 0)
 			(effects
@@
 			)
 		)
-		(property "Footprint" "Capacitor_THT:CP_Radial_D6.3mm_P2.50mm"
+		(property "Footprint" "values_not_refs:CP_Radial_D8.0mm_P2.50mm_VALUE"
 			(at 157.48 91.44 0)
 			(effects
@@
 			)
 		)
-		(property "Footprint" "Capacitor_THT:CP_Radial_D5.0mm_P2.50mm"
+		(property "Footprint" "values_not_refs:CP_Radial_D6.3mm_P2.50mm_VALUE"
 			(at 127 91.44 0)
 			(effects
@@
 			)
 		)
-		(property "Footprint" "Capacitor_THT:CP_Radial_D5.0mm_P2.50mm"
+		(property "Footprint" "values_not_refs:CP_Radial_D6.3mm_P2.50mm_VALUE"
 			(at 127 102.87 0)
 			(effects
