File: hardware/iosefka_motherboard/iosefka_motherboard.kicad_pcb (KiCad board)
At the start: 2 copper layers, 213 x 128.5 mm, 123 parts, among them J1 Audio Out, J2 DC In, J3 Audio In, J4 Conn_01x10, J5 Conn_01x10, J6 Conn_01x10, J7 Conn_01x08, J8 Conn_01x08, J9 Conn_01x10, Q1 2N3906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

Commit message: parameter adjustments
Parts:
- added REF**: MountingHole_3.2mm_M3_DIN965_Pad, MountingHole:MountingHole_3.2mm_M3_DIN965_Pad, F.Cu at (153.4, 132.6)
- C1, C16, C20, C9: footprint Capacitor_THT:CP_Radial_D5.0mm_P2.50mm -> values_not_refs:CP_Radial_D6.3mm_P2.50mm_VALUE
- C15, C25, C30, C36, C8: value 4.7u BP -> 4.7u NP; footprint Capacitor_THT:CP_Radial_D5.0mm_P2.50mm -> values_not_refs:CP_Radial_D6.3mm_P2.50mm_VALUE
- C17, C2: footprint Capacitor_THT:CP_Radial_D6.3mm_P2.50mm -> values_not_refs:CP_Radial_D8.0mm_P2.50mm_VALUE
- Q1, Q2: footprint Package_TO_SOT_THT:TO-92_Inline_Wide -> values_not_refs:TO-92_Inline_Wide
- R27: value 1M -> DNP
- R35, R37: value 30k -> 15k
- R36: value 15k -> 7.5k
- moved C16 1.99 mm to (137.0, 82.8)
- moved C19 1.99 mm to (118.0, 82.8)
- moved C20 1.23 mm to (118.1, 75.1)
- moved C1 1.23 mm to (134.6, 75.1)
- moved C25 0.53 mm to (247.6, 75.7)
Routing:
- net Net-(U2-VI): track 43.6 -> 41.6 mm
- net Net-(D3-K): track 96.3 -> 97.8 mm
- net IN_MIX: track 170.5 -> 171.5 mm
- net Net-(C25-Pad2): track 4.95 -> 5.66 mm
- net Net-(U3-CAP+): track 19.5 -> 18.8 mm
- net DELAY_IN: track 68.9 -> 69.6 mm
- net Net-(C25-Pad1): track 106.3 -> 105.7 mm
Other:
- board text added: "2026 Global Sequence Iosefka Motherboard v1.3"
- board text removed: "2025 Global Sequence Iosefka Motherboard v1.2"

Commit message: added docs
Connections:
- J9 pad 6: PIN_ENCODER_A -> PIN_ENCODER_B
- J9 pad 7: PIN_ENCODER_B -> PIN_ENCODER_A
- U6 pad 19: PIN_ENCODER_A -> PIN_ENCODER_B
- U6 pad 20: PIN_ENCODER_B -> PIN_ENCODER_A
Routing:
- net PIN_ENCODER_B: track 74.6 -> 75.2 mm, vias 1 -> 0
- net PIN_ENCODER_A: track 75.2 -> 74.6 mm, vias 0 -> 1
