File: hardware/iosefka_bottomboard/iosefka_bottomboard.kicad_pcb (KiCad board)
At the start: 2 copper layers, 213 x 128.5 mm, 2 parts

Commit message: parameter adjustments
Parts:
- added REF**: MountingHole_3.2mm_M3_DIN965_Pad, MountingHole:MountingHole_3.2mm_M3_DIN965_Pad, F.Cu at (153.9, 122.4)
Other:
- board text added: "2025 Global Sequence | https://github.com/globalsequence"
- board text removed: "2025 Global Sequence https://github.com/globalsequence"

Commit message: added docs
Other:
- board text added: "2026 Global Sequence | https://github.com/globalsequence"
- board text removed: "2025 Global Sequence | https://github.com/globalsequence"
Changed lines of the file:
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@@
 		(layer "Edge.Cuts")
 	)
-	(gr_text "2025 Global Sequence | https://github.com/globalsequence"
+	(gr_text "2026 Global Sequence | https://github.com/globalsequence"
 		(at 117.87381 151.414992 0)
 		(layer "B.SilkS")
@@
 			(justify left bottom mirror)
 		)
-		(render_cache "2025 Global Sequence | https://github.com/globalsequence"
+		(render_cache "2026 Global Sequence | https://github.com/globalsequence"
 			0
 			(polygon
@@
 			(polygon
 				(pts
-					(xy 113.341151 149.702686) (xy 114.162265 149.702686) (xy 114.305055 150.51116) (xy 114.038342 150.51116)
-					(xy 114.011631 150.47573) (xy 113.981892 150.446377) (xy 113.951088 150.424271) (xy 113.91759 150.40756)
-					(xy 113.843498 150.390395) (xy 113.817882 150.389344) (xy 113.772874 150.392274) (xy 113.731701 150.401056)
-					(xy 113.696669 150.414562) (xy 113.665009 150.433174) (xy 113.630945 150.4628) (xy 113.607592 150.491864)
-					(xy 113.58901 150.524417) (xy 113.566126 150.600352) (xy 113.56161 150.660271) (xy 113.564541 150.708577)
-					(xy 113.573334 150.753198) (xy 113.58695 150.791788) (xy 113.605748 150.827105) (xy 113.633051 150.86287)
-					(xy 113.661431 150.88978) (xy 113.692648 150.911091) (xy 113.761041 150.936398) (xy 113.815776 150.941638)
-					(xy 113.857829 150.938708) (xy 113.89671 150.929923) (xy 113.930616 150.916204) (xy 113.961674 150.89724)
-					(xy 113.98064 150.881829) (xy 114.006316 150.854596) (xy 114.026932 150.824024) (xy 114.052697 150.754086)
-					(xy 114.05721 150.7253) (xy 114.351217 150.7253) (xy 114.344773 150.787178) (xy 114.332701 150.844767)
-					(xy 114.316098 150.895301) (xy 114.294457 150.941991) (xy 114.26872 150.983507) (xy 114.238267 151.021418)
-					(xy 114.192673 151.064462) (xy 114.149593 151.095732) (xy 114.10309 151.122231) (xy 113.999215 151.161076)
-					(xy 113.878008 151.180895) (xy 113.815776 151.183164) (xy 113.749227 151.180233) (xy 113.686143 151.171442)
-					(xy 113.62903 151.157548) (xy 113.575086 151.138293) (xy 113.52554 151.11436) (xy 113.479004 151.085334)
-					(xy 113.416713 151.034054) (xy 113.378267 150.993111) (xy 113.345281 150.949286) (xy 113.318317 150.903675)
-					(xy 113.296565 150.855316) (xy 113.268671 150.750242) (xy 113.261375 150.653951) (xy 113.264306 150.590436)
-					(xy 113.273099 150.530759) (xy 113.286864 150.477678) (xy 113.305909 150.428056) (xy 113.329411 150.383256)
-					(xy 113.357875 150.341711) (xy 113.389419 150.305355) (xy 113.426615 150.271177) (xy 113.46704 150.242091)
-					(xy 113.556201 150.199675) (xy 113.659441 150.176896) (xy 113.72968 150.173006) (xy 113.784497 150.175937)
-					(xy 113.835599 150.184726) (xy 113.880506 150.198424) (xy 113.922101 150.217357) (xy 113.993654 150.269276)
-					(xy 114.000515 150.275955) (xy 113.94382 149.95676) (xy 113.341151 149.95676)
+					(xy 113.812528 149.682444) (xy 113.871193 149.691237) (xy 113.924381 149.705157) (xy 113.974624 149.724457)
+					(xy 114.020962 149.748564) (xy 114.064474 149.777829) (xy 114.143296 149.852147) (xy 114.170691 149.886418)
+					(xy 114.233733 149.991205) (xy 114.281098 150.11617) (xy 114.311855 150.264984) (xy 114.323861 150.442035)
+					(xy 114.323923 150.456572) (xy 114.320992 150.550771) (xy 114.312199 150.638909) (xy 114.29859 150.71623)
+					(xy 114.2798 150.788193) (xy 114.257219 150.851435) (xy 114.229987 150.909865) (xy 114.176919 150.993113)
+					(xy 114.140282 151.036157) (xy 114.100429 151.073755) (xy 114.058737 151.104993) (xy 114.01402 151.131111)
+					(xy 113.916167 151.167815) (xy 113.804133 151.184396) (xy 113.769522 151.185271) (xy 113.706495 151.18234)
+					(xy 113.646691 151.173547) (xy 113.592407 151.159621) (xy 113.541085 151.140311) (xy 113.493732 151.116205)
+					(xy 113.449218 151.086944) (xy 113.392625 151.038267) (xy 113.355713 150.997499) (xy 113.324171 150.953805)
+					(xy 113.298465 150.908133) (xy 113.277917 150.85965) (xy 113.252215 150.753702) (xy 113.247139 150.670712)
+					(xy 113.536423 150.670712) (xy 113.539353 150.718055) (xy 113.54814 150.761928) (xy 113.561818 150.800191)
+					(xy 113.580714 150.835357) (xy 113.603651 150.866076) (xy 113.631091 150.893301) (xy 113.661225 150.914678)
+					(xy 113.692559 150.929646) (xy 113.726356 150.939259) (xy 113.773735 150.943745) (xy 113.812806 150.940814)
+					(xy 113.848949 150.932021) (xy 113.880567 150.918237) (xy 113.909527 150.899161) (xy 113.941713 150.868182)
+					(xy 113.964508 150.83719) (xy 113.982411 150.802896) (xy 114.003605 150.723935) (xy 114.006835 150.672819)
+					(xy 114.003904 150.624724) (xy 113.995111 150.58023) (xy 113.981463 150.541592) (xy 113.962612 150.506134)
+					(xy 113.941713 150.477546) (xy 113.915107 150.450277) (xy 113.885788 150.42889) (xy 113.855266 150.413952)
+					(xy 113.822277 150.404361) (xy 113.775842 150.399877) (xy 113.736235 150.402808) (xy 113.69951 150.411601)
+					(xy 113.667243 150.425412) (xy 113.637593 150.444531) (xy 113.603651 150.476539) (xy 113.580067 150.507844)
+					(xy 113.561554 150.54226) (xy 113.539791 150.620145) (xy 113.536423 150.670712) (xy 113.247139 150.670712)
+					(xy 113.246629 150.662377) (xy 113.24956 150.60018) (xy 113.258352 150.541414) (xy 113.272214 150.488521)
+					(xy 113.291417 150.438758) (xy 113.3153 150.393226) (xy 113.344268 150.350676) (xy 113.375772 150.313782)
+					(xy 113.413751 150.277886) (xy 113.454633 150.247454) (xy 113.497308 150.22303) (xy 113.542745 150.203806)
+					(xy 113.642253 150.180909) (xy 113.706599 150.177219) (xy 113.759786 150.18015) (xy 113.810019 150.188943)
+					(xy 113.855354 150.202859) (xy 113.897973 150.222152) (xy 113.974076 150.275981) (xy 114.034129 150.343182)
+					(xy 114.024261 150.252881) (xy 114.009317 150.173028) (xy 113.991646 150.11044) (xy 113.969915 150.056214)
+					(xy 113.946913 150.014601) (xy 113.920631 149.979744) (xy 113.893577 149.953659) (xy 113.863751 149.933283)
+					(xy 113.79857 149.910133) (xy 113.754868 149.906385) (xy 113.715538 149.909316) (xy 113.680216 149.918112)
+					(xy 113.651143 149.931454) (xy 113.625496 149.949808) (xy 113.584973 150.000683) (xy 113.557489 150.072256)
+					(xy 113.273923 150.072256) (xy 113.285535 150.013141) (xy 113.302413 149.95855) (xy 113.323287 149.910957)
+					(xy 113.3489 149.867438) (xy 113.378326 149.829061) (xy 113.41223 149.794532) (xy 113.426239 149.782462)
+					(xy 113.465933 149.753552) (xy 113.50908 149.729393) (xy 113.606429 149.695171) (xy 113.721646 149.680073)
+					(xy 113.750654 149.679513)
 				)
 			)
