File: hardware/iosefka_controlboard/components_and_display.kicad_sch (KiCad schematic)
At the start: 47 parts, among them SW1 RotaryEncoder_Switch, SW10 SW_Push, SW11 SW_Push, SW12 SW_Push, SW13 SW_Push, SW14 SW_Push, SW15 SW_Push, SW16 SW_Push, SW17 SW_Push, SW18 SW_Push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

Commit message: added docs
Connections:
- net PIN_ENCODER_A: now also SW1.A; no longer SW1.B
- net PIN_ENCODER_B: now also SW1.B; no longer SW1.A
Changed lines of the file:
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@@
 		)
 	)
-	(global_label "PIN_ENCODER_A"
+	(global_label "PIN_ENCODER_B"
 		(shape output)
 		(at 48.26 58.42 0)
@@
 		)
 		(property "Intersheetrefs" "${INTERSHEET_REFS}"
-			(at 66.2433 58.42 0)
+			(at 66.4247 58.42 0)
 			(effects
 				(font
@@
 		)
 	)
-	(global_label "PIN_ENCODER_B"
+	(global_label "PIN_ENCODER_A"
 		(shape output)
 		(at 40.64 58.42 180)
@@
 		)
 		(property "Intersheetrefs" "${INTERSHEET_REFS}"
-			(at 22.4753 58.42 0)
+			(at 22.6567 58.42 0)
 			(effects
 				(font
