File: hardware/iosefka_controlboard/iosefka_controlboard.kicad_pcb (KiCad board)
At the start: 2 copper layers, 213 x 128.5 mm, 77 parts, among them J1 Conn_01x10, J2 Conn_01x10, J3 DIN-5_180degree, J6 DIN-5_180degree, SW1 RotaryEncoder_Switch, SW10 SW_Push, SW11 SW_Push, SW12 SW_Push, SW13 SW_Push, SW14 SW_Push, SW15 SW_Push, SW16 SW_Push, SW17 SW_Push, SW18 SW_Push, SW19 SW_Push, SW2 SW_Push, SW20 SW_Push, SW21 SW_Push, SW3 SW_Push, SW4 SW_Push, SW5 SW_Push, SW6 SW_Push, SW7 SW_Push, SW8 SW_Push, SW9 SW_Push, U1 SSD1306_SPI, U14 H11L1, U2 MCP23017_SP, U3 MCP23017_SP, U4 4051, U5 4051

Commit message: updated settings
Other:
- board text added: "2025 Global Sequence Iosefka Control Board v1.1"
- board text added: "Osc 1"
- board text added: "Osc 2"
- board text added: "User"
- board text removed: "2025 Global Sequence Iosefka Control Board v1.0"

Commit message: parameter adjustments
Parts:
- added REF**: MountingHole_3.2mm_M3_DIN965_Pad, MountingHole:MountingHole_3.2mm_M3_DIN965_Pad, F.Cu at (157.7, 133.8)
- R2, R3, R4, R5, R6, R7, R8, R9: moved to B.Cu
- U1: footprint SSD1306:128x64_0.96_Disp_Module -> SSD1306 SPI:128x64_0.96_Disp_Module_oval_holes
Routing:
- net PIN_DISPLAY_SCK: track 45.7 -> 50.5 mm
- net PIN_DISPLAY_MOSI: track 47.8 -> 52.4 mm
- net PIN_DISPLAY_DC: track 53.9 -> 56.9 mm
- net SW_B_1: track 126.3 -> 123.6 mm
- net SW_A_8: track 161.2 -> 158.9 mm
- net SW_A_6: track 120.4 -> 118.0 mm
- net SW_A_7: track 140.8 -> 138.4 mm
- net PIN_DISPLAY_CS: track 57.5 -> 58.8 mm
- net LED_8: track 113.1 -> 114.2 mm
- net +3.3V: track 730.0 -> 731.0 mm
- net LED_6: track 79.7 -> 80.6 mm
- net LED_7: track 62.1 -> 62.7 mm
Other:
- board text added: "2026 Global Sequence Iosefka Control Board v1.2"
- board text added: "7.5v - 9v"
- board text added: "BRR"
- board text added: "Clear All"
- board text added: "Copy Step"
- board text added: "D. Input"
- board text added: "D. Type"
- board text added: "DC In"
- board text added: "Gen New"
- board text added: "Gen On/Off"
- board text added: "Loop"
- board text added: "Mix O1"
- board text added: "Mix O2"
- board text added: "Record"
- board text added: "SRR"
- board text added: "Section +"
- board text added: "Section -"
- board text removed: "2025 Global Sequence Iosefka Control Board v1.1"
- board text removed: "DC In 7.5v - 9v"
- board text removed: "Generate New"
- board text removed: "Generator On/Off"
- board text removed: "Mix 1"
- board text removed: "Mix 2"
- board text removed: "Section Down"
- board text removed: "Section Up"
- board text removed: "Synth + Env"

Commit message: added docs
Connections:
- J2 pad 6: PIN_ENCODER_A -> PIN_ENCODER_B
- J2 pad 7: PIN_ENCODER_B -> PIN_ENCODER_A
- SW1 pad A: PIN_ENCODER_B -> PIN_ENCODER_A
- SW1 pad B: PIN_ENCODER_A -> PIN_ENCODER_B
Routing:
- net PIN_ENCODER_B: track 20.5 -> 27.0 mm
- net PIN_ENCODER_A: track 27.0 -> 20.5 mm
Other:
- board text added: "G. Chance"
- board text added: "Probability"
- board text removed: "G. Mode"
- board text removed: "Probability/G. Chance"
